Commit message: fix: Remove comment from inertia macro file
* Note all of inertia is correct, but there a small issue that is is for main body it dont include 0.1 z axis in origin

File: learn_ros/description/urdf/inertials.urdf.xacro (robot description, xacro)
@@ -1,3 +1,2 @@
-<!-- Source of formulas: https://en.wikipedia.org/wiki/List_of_moments_of_inertia -->
 <?xml version="1.0"?>
 <robot name="inertial_macros" xmlns:xacro="http://www.ros.org/wiki/xacro">

File: learn_ros/description/urdf/robot.urdf.xacro (robot description, xacro)
@@ -58,5 +58,5 @@
             <origin xyz="0 0 0.1" rpy="0 0 0" />
         </collision>
-        <xacro:solid_box_inertia mass="5" x="0.6" y="0.4" z="0.2"/>
+        <xacro:solid_box_inertia mass="5" x="0.6" y="0.4" z="0.2" />
     </link>
     <link name="lidar_link">
@@ -68,4 +68,10 @@
             <material name="white" />
         </visual>
+        <collision>
+            <geometry>
+                <box size="${radius*2} ${radius*2} ${length}" />
+            </geometry>
+            <origin xyz="0 0 0" rpy="0 0 0" />
+        </collision>
     </link>
     <link name="caster_wheel_link">

Commit message: fix: Update inertia macros to include position and orientation parameters
- This is to fix origin position error from previous commit when calc inertia

File: learn_ros/description/urdf/inertials.urdf.xacro (robot description, xacro)
@@ -1,6 +1,7 @@
 <?xml version="1.0"?>
 <robot name="inertial_macros" xmlns:xacro="http://www.ros.org/wiki/xacro">
-    <xacro:macro name="solid_box_inertia" params="mass x y z">
+    <xacro:macro name="solid_box_inertia" params="mass x y z xyz:='0 0 0' rpy:='0 0 0'">
         <inertial>
+            <origin xyz="${xyz}" rpy="${rpy}" />
             <mass value="${mass}"/>
             <inertia
@@ -10,6 +11,7 @@
         </inertial>
     </xacro:macro>
-    <xacro:macro name="solid_cylinder_inertia" params="mass radius length">
+    <xacro:macro name="solid_cylinder_inertia" params="mass radius length xyz:='0 0 0' rpy:='0 0 0'">
         <inertial>
+            <origin xyz="${xyz}" rpy="${rpy}" />
             <mass value="${mass}"/>
             <inertia
@@ -19,6 +21,7 @@
         </inertial>
     </xacro:macro>
-    <xacro:macro name="solid_sphere_inertia" params="mass radius">
+    <xacro:macro name="solid_sphere_inertia" params="mass radius xyz:='0 0 0' rpy:='0 0 0'">
         <inertial>
+            <origin xyz="${xyz}" rpy="${rpy}" />
             <mass value="${mass}"/>
             <inertia

File: learn_ros/description/urdf/robot.urdf.xacro (robot description, xacro)
@@ -23,5 +23,7 @@
                 <origin xyz="0 0 0" rpy="1.57 0 0" />
             </collision>
-            <xacro:solid_cylinder_inertia mass="0.5" radius="${radius}" length="${length}"/>
+            <xacro:solid_cylinder_inertia
+                mass="0.5" radius="${radius}" length="${length}"
+                xyz="0 0 0" rpy="1.57 0 0" />
         </link>
     </xacro:macro>
@@ -58,5 +60,7 @@
             <origin xyz="0 0 0.1" rpy="0 0 0" />
         </collision>
-        <xacro:solid_box_inertia mass="5" x="0.6" y="0.4" z="0.2" />
+        <xacro:solid_box_inertia
+            mass="5" x="0.6" y="0.4" z="0.2"
+            xyz="0 0 0.1" rpy="0 0 0"/>
     </link>
     <link name="lidar_link">
