Commit message: feat: Sync sensor data gz and rviz2

File: learn_ros_description/urdf/sensors/camera.xacro (robot description, xacro)
@@ -16,8 +16,14 @@
     </collision>
   </link>
+  <link name="camera_optical_link"></link>
   <joint name="camera_joint" type="fixed">
     <parent link="base_link" />
     <child link="camera_link" />
     <origin xyz="0.3125 0 0.1" rpy="0 0 0" />
+  </joint>
+  <joint name="camera_optical_joint" type="fixed">
+    <parent link="camera_link" />
+    <child link="camera_optical_link" />
+    <origin xyz="0 0 0.3" rpy="${-pi/2} 0 ${-pi/2}" />
   </joint>
   <gazebo reference="camera_link">
@@ -41,4 +47,5 @@
         </clip>
       </camera>
+      <gz_frame_id>camera_optical_link</gz_frame_id>
     </sensor>
   </gazebo>

File: learn_ros_description/urdf/sensors/lidar.xacro (robot description, xacro)
@@ -50,4 +50,5 @@
         </noise>
       </lidar>
+      <gz_frame_id>lidar_link</gz_frame_id>
     </sensor>
   </gazebo>
