Commit message: feat: Sync gazebo and rviz2 in term of move

File: learn_ros_description/urdf/robot.urdf.xacro (robot description, xacro)
@@ -6,5 +6,10 @@
   <xacro:include filename="$(find learn_ros_description)/urdf/body/wheels.xacro" />
   <xacro:include filename="$(find learn_ros_description)/urdf/body/caster_wheel.xacro" />
-  <link name="world_ground" />
+  <link name="base_footprint"/>
+  <joint name="base_footprint_joint" type="fixed">
+    <parent link="base_footprint"/>
+    <child link="base_link"/>
+    <origin xyz="0 0 0.1" rpy="0 0 0"/>
+  </joint>
   <link name="base_link">
     <visual>
@@ -25,9 +30,4 @@
       xyz="0 0 0.1" rpy="0 0 0"/>
   </link>
-  <joint name="base_joint" type="fixed">
-    <parent link="world_ground" />
-    <child link="base_link" />
-    <origin xyz="0 0 0.1" rpy="0 0 0" />
-  </joint>
   <gazebo>
     <plugin
@@ -39,6 +39,19 @@
       <wheel_radius>${wheels_radius}</wheel_radius>
       <topic>cmd_vel</topic>
+      <odom_topic>odom</odom_topic>
+      <tf_topic>/tf</tf_topic>
+      <frame_id>odom</frame_id>
+      <child_frame_id>base_footprint</child_frame_id>
     </plugin>
   </gazebo>
+  <gazebo>
+  <plugin
+    filename="gz-sim-joint-state-publisher-system"
+    name="gz::sim::systems::JointStatePublisher">
+    <topic>/model/my_robot/joint_state</topic>
+    <joint_name>left_wheel_joint</joint_name>
+    <joint_name>right_wheel_joint</joint_name>
+  </plugin>
+</gazebo>
   <gazebo>
     <plugin
@@ -48,9 +61,3 @@
     </plugin>
   </gazebo>
-  <gazebo>
-    <plugin
-      filename="gz-sim-joint-state-publisher-system"
-      name="gz::sim::systems::JointStatePublisher">
-    </plugin>
-  </gazebo>
 </robot>

Commit message: feat: Re-enable camera sensor

File: learn_ros_description/urdf/robot.urdf.xacro (robot description, xacro)
@@ -3,5 +3,5 @@
   <xacro:include filename="$(find learn_ros_description)/urdf/commons.xacro" />
   <xacro:include filename="$(find learn_ros_description)/urdf/sensors/lidar.xacro" />
-  <!-- <xacro:include filename="$(find learn_ros_description)/urdf/sensors/camera.xacro" /> -->
+  <xacro:include filename="$(find learn_ros_description)/urdf/sensors/camera.xacro" />
   <xacro:include filename="$(find learn_ros_description)/urdf/body/wheels.xacro" />
   <xacro:include filename="$(find learn_ros_description)/urdf/body/caster_wheel.xacro" />

File: learn_ros_description/urdf/sensors/camera.xacro (robot description, xacro)
@@ -25,5 +25,5 @@
     <parent link="camera_link" />
     <child link="camera_optical_link" />
-    <origin xyz="0 0 0.3" rpy="${-pi/2} 0 ${-pi/2}" />
+    <origin xyz="0 0 0" rpy="${-pi/2} 0 ${-pi/2}" />
   </joint>
   <gazebo reference="camera_link">
